Commit message: Made a package contains hc1- and idec cad files. You can run a demo with roslaunch hc10_idec_moveit config demo.launch

File: motoman_hc10_description/urdf/hc10_macro.xacro (robot description, xacro)
@@ -8,5 +8,13 @@
     </inertial>
   </xacro:macro>
-  <xacro:macro name="motoman_hc10" params="prefix">
+  <xacro:macro name="motoman_hc10" params="prefix parent *origin
+    joint_1_s_lower_limit:=${-pi}    joint_1_s_upper_limit:=${pi}
+    joint_2_l_lower_limit:=${-pi}    joint_2_l_upper_limit:=${pi}
+    joint_3_u_lower_limit:=${-pi}    joint_3_u_upper_limit:=${pi}
+    joint_4_r_lower_limit:=${-pi}    joint_4_r_upper_limit:=${pi}
+    joint_5_b_lower_limit:=${-pi}    joint_5_b_upper_limit:=${pi}
+    joint_6_t_lower_limit:=${-pi}    joint_6_t_upper_limit:=${pi}
+    safety_limits:=false safety_pos_margin:=${radians(10.0)}
+    safety_k_position:=20">
     <!-- Properties -->
     <material name="yaskawa_blue">
@@ -116,4 +124,10 @@
     <!-- end of link list -->
     <!-- joint list -->
+    <joint name="${prefix}joint_base" type="fixed">
+      <parent link="${parent}"/>
+      <child link="${prefix}base_link"/>
+      <xacro:insert_block name="origin"/>
+      <axis xyz="0 0 1" />
+    </joint>
     <joint name="${prefix}joint_1_s" type="revolute">
       <parent link="${prefix}base_link"/>
@@ -122,4 +136,8 @@
       <axis xyz="0 0 1" />
       <limit lower="${radians(-180)}" upper="${radians(180)}" effort="368.48" velocity="${radians(130)}"/>
+      <xacro:if value="${safety_limits}">
+        <safety_controller soft_lower_limit="${joint_1_s_lower_limit + safety_pos_margin}" soft_upper_limit="${joint_1_s_upper_limit - safety_pos_margin}" k_position="${safety_k_position}" k_velocity="0.0"/>
+      </xacro:if>
+      <dynamics damping="0.0" friction="0.0"/>
     </joint>
     <joint name="${prefix}joint_2_l" type="revolute">
@@ -129,11 +147,17 @@
       <axis xyz="0 1 0" />
       <limit lower="${radians(-180)}" upper="${radians(180)}" effort="368.48" velocity="${radians(130)}"/>
+      <xacro:if value="${safety_limits}">
+        <safety_controller soft_lower_limit="${joint_2_l_lower_limit + safety_pos_margin}" soft_upper_limit="${joint_2_l_upper_limit - safety_pos_margin}" k_position="${safety_k_position}" k_velocity="0.0"/>
+      </xacro:if>
     </joint>
     <joint name="${prefix}joint_3_u" type="revolute">
       <parent link="${prefix}link_2_l"/>
       <child link="${prefix}link_3_u"/>
-      <origin xyz="0 0 0.700" rpy="0 0 0" />
+      <origin xyz="0 0 0.700" rpy="0 0  0" />
       <axis xyz="0 -1 0" />
       <limit lower="${radians(-5)}" upper="${radians(355)}" effort="141.12" velocity="${radians(180)}"/>
+      <xacro:if value="${safety_limits}">
+        <safety_controller soft_lower_limit="${joint_3_u_lower_limit + safety_pos_margin}" soft_upper_limit="${joint_3_u_upper_limit - safety_pos_margin}" k_position="${safety_k_position}" k_velocity="0.0"/>
+      </xacro:if>
     </joint>
     <joint name="${prefix}joint_4_r" type="revolute">
@@ -143,4 +167,7 @@
       <axis xyz="0 0 1" />
       <limit lower="${radians(-180)}" upper="${radians(180)}" effort="39.20" velocity="${radians(180)}"/>
+      <xacro:if value="${safety_limits}">
+        <safety_controller soft_lower_limit="${joint_4_r_lower_limit + safety_pos_margin}" soft_upper_limit="${joint_4_r_upper_limit - safety_pos_margin}" k_position="${safety_k_position}" k_velocity="0.0"/>
+      </xacro:if>
     </joint>
     <joint name="${prefix}joint_5_b" type="revolute">
@@ -150,4 +177,7 @@
       <axis xyz="0 -1 0" />
       <limit lower="${radians(-180)}" upper="${radians(180)}" effort="31.36" velocity="${radians(250)}"/>
+      <xacro:if value="${safety_limits}">
+        <safety_controller soft_lower_limit="${joint_5_b_lower_limit + safety_pos_margin}" soft_upper_limit="${joint_5_b_upper_limit - safety_pos_margin}" k_position="${safety_k_position}" k_velocity="0.0"/>
+      </xacro:if>
     </joint>
     <joint name="${prefix}joint_6_t" type="revolute">
@@ -157,4 +187,7 @@
       <axis xyz="0 0 1" />
       <limit lower="${radians(-180)}" upper="${radians(180)}" effort="31.36" velocity="${radians(250)}"/>
+      <xacro:if value="${safety_limits}">
+        <safety_controller soft_lower_limit="${joint_6_t_lower_limit + safety_pos_margin}" soft_upper_limit="${joint_6_t_upper_limit - safety_pos_margin}" k_position="${safety_k_position}" k_velocity="0.0"/>
+      </xacro:if>
     </joint>
     <joint name="${prefix}joint_6_t-tool0" type="fixed">

File: motoman_hc10_description/urdf/hc10_robot.urdf.xacro (robot description, xacro)
@@ -4,4 +4,5 @@
   <xacro:arg name="prefix" default=""/>
   <xacro:include filename="$(find motoman_hc10_description)/urdf/common.gazebo.xacro" />
+  <link name="world" />
   <!-- transimission -->
   <xacro:include filename="$(find motoman_hc10_description)/urdf/hc10.transmission.xacro" />
@@ -11,10 +12,6 @@
   <!-- hc10 -->
   <xacro:include filename="$(find motoman_hc10_description)/urdf/hc10_macro.xacro" />
-  <xacro:motoman_hc10 prefix="$(arg prefix)"/>
-  <link name="world" />
-  <joint name="world_joint" type="fixed">
-    <parent link="world" />
-    <child link = "base_link" />
-    <origin xyz="0.0 0.0 0.0" rpy="0.0 0.0 0.0" />
-  </joint>
+  <xacro:motoman_hc10 prefix="$(arg prefix)" parent="world">
+    <origin xyz="0 0 0" rpy="0 0 0" />
+  </xacro:motoman_hc10>
 </robot>
